File: PCB/V5/BL706 Robot.kicad_pcb (KiCad board)
At the start: 2 copper layers, 104.8 x 60.4 mm, 86 parts, among them J1 Conn_01x04_Male, M1 Conn_01x02_Male, M2 Conn_01x02_Male, SW2 SW_SPST, U1 BL706C, U2 FM8002A, U3 TC8301, U4 TC8301, Y1 32MHz

Commit message: updated last file
Parts:
- removed the G*** at (179.1, 132.7)
- removed the G*** at (199.8, 132.2)
- removed the G*** at (221.3, 124.4)
- D5: value 1N4728A -> ZM4728A; footprint Diode_THT:D_DO-41_SOD81_P3.81mm_Vertical_KathodeUp -> Diode_SMD:D_MELF
- moved D5 2.32 mm to (222.6, 120.7)
- moved SW2 0.32 mm to (221.5, 112.3), turned to 160 degrees
- renumbered BOOT to BOOT1, RST to RST1
Routing:
- net /S_SD: track 91.9 -> 92.8 mm
- net /MOTOR2A: track 25.4 -> 24.7 mm
- net /M_VCC: track 95.9 -> 96.4 mm
- net /MOTOR1A: track 40.9 -> 40.4 mm
- net /MOTOR2B: track 26.8 -> 26.2 mm
- net VCC: vias 10 -> 11
Other:
- outline, holes or cut-outs redrawn
- board text added: "Line Following Robot V5"
- board text removed: "Line Following Robt V5"
