File: PCB/V5/BL706 Robot.kicad_sch (KiCad schematic)
At the start: 81 parts, among them J1 Conn_01x04_Male, M1 Conn_01x02_Male, M2 Conn_01x02_Male, SW2 SW_SPST, U1 BL706C, U2 FM8002A, U3 TC8301, U4 TC8301, Y1 32MHz

Commit message: updated last file
Parts:
- D5: value 1N4728A -> ZM4728A; footprint Diode_THT:D_DO-41_SOD81_P3.81mm_Vertical_KathodeUp -> Diode_SMD:D_MELF; LCSC C261315 -> C38989
- SW2: LCSC C431541 -> C319019
Other:
- moved on the sheet: AE1, C4, C6, L2
Changed lines of the file:
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@@
   (junction (at 185.42 25.4) (diameter 0) (color 0 0 0 0)
   )
-  (junction (at 115.57 152.4) (diameter 0) (color 0 0 0 0)
+  (junction (at 121.92 132.08) (diameter 0) (color 0 0 0 0)
   )
   (junction (at 80.01 127) (diameter 0) (color 0 0 0 0)
@@
   (junction (at 62.23 127) (diameter 0) (color 0 0 0 0)
   )
-  (junction (at 134.62 152.4) (diameter 0) (color 0 0 0 0)
+  (junction (at 140.97 132.08) (diameter 0) (color 0 0 0 0)
   )
   (junction (at 96.52 34.29) (diameter 0) (color 0 0 0 0)
@@
     (stroke (width 0) (type default) (color 0 0 0 0))
   )
-  (wire (pts (xy 129.54 152.4) (xy 134.62 152.4))
+  (wire (pts (xy 135.89 132.08) (xy 140.97 132.08))
     (stroke (width 0) (type default) (color 0 0 0 0))
   )
-  (wire (pts (xy 106.68 152.4) (xy 115.57 152.4))
+  (wire (pts (xy 113.03 132.08) (xy 121.92 132.08))
     (stroke (width 0) (type default) (color 0 0 0 0))
   )
@@
     (stroke (width 0) (type default) (color 0 0 0 0))
   )
-  (wire (pts (xy 115.57 152.4) (xy 115.57 156.21))
+  (wire (pts (xy 121.92 132.08) (xy 121.92 135.89))
     (stroke (width 0) (type default) (color 0 0 0 0))
   )
@@
     (stroke (width 0) (type default) (color 0 0 0 0))
   )
-  (wire (pts (xy 134.62 152.4) (xy 139.7 152.4))
+  (wire (pts (xy 140.97 132.08) (xy 146.05 132.08))
     (stroke (width 0) (type default) (color 0 0 0 0))
   )
@@
     (stroke (width 0) (type default) (color 0 0 0 0))
   )
-  (wire (pts (xy 134.62 152.4) (xy 134.62 156.21))
+  (wire (pts (xy 140.97 132.08) (xy 140.97 135.89))
     (stroke (width 0) (type default) (color 0 0 0 0))
   )
@@
     (stroke (width 0) (type default) (color 0 0 0 0))
   )
-  (wire (pts (xy 121.92 152.4) (xy 115.57 152.4))
+  (wire (pts (xy 128.27 132.08) (xy 121.92 132.08))
     (stroke (width 0) (type default) (color 0 0 0 0))
   )
@@
     (effects (font (size 1.27 1.27)) (justify left bottom))
   )
-  (label "ANT" (at 134.62 152.4 0)
+  (label "ANT" (at 140.97 132.08 0)
     (effects (font (size 1.27 1.27)) (justify left bottom))
   )
@@
     (pin "2")
   )
-  (symbol (lib_id "Device:L") (at 125.73 152.4 90) (unit 1)
+  (symbol (lib_id "Device:L") (at 132.08 132.08 90) (unit 1)
     (in_bom yes) (on_board yes)
-    (property "Reference" "L2" (id 0) (at 125.73 149.86 90))
-    (property "Value" "2.7nH" (id 1) (at 125.73 153.67 90))
-    (property "Footprint" "Inductor_SMD:L_0402_1005Metric" (id 2) (at 125.73 152.4 0)
+    (property "Reference" "L2" (id 0) (at 132.08 129.54 90))
+    (property "Value" "2.7nH" (id 1) (at 132.08 133.35 90))
+    (property "Footprint" "Inductor_SMD:L_0402_1005Metric" (id 2) (at 132.08 132.08 0)
       (effects (font (size 1.27 1.27)) hide)
     )
-    (property "Datasheet" "~" (id 3) (at 125.73 152.4 0)
+    (property "Datasheet" "~" (id 3) (at 132.08 132.08 0)
       (effects (font (size 1.27 1.27)) hide)
     )
-    (property "LCSC PN" "" (id 4) (at 125.73 152.4 90)
+    (property "LCSC PN" "" (id 4) (at 132.08 132.08 90)
       (effects (font (size 1.27 1.27)) hide)
     )
@@
     (pin "1")
   )
-  (symbol (lib_id "Device:C") (at 134.62 160.02 0) (unit 1)
+  (symbol (lib_id "Device:C") (at 140.97 139.7 0) (unit 1)
     (in_bom yes) (on_board yes)
-    (property "Reference" "C6" (id 0) (at 137.16 158.75 0)
+    (property "Reference" "C6" (id 0) (at 143.51 138.43 0)
       (effects (font (size 1.27 1.27)) (justify left))
     )
-    (property "Value" "2.7pF" (id 1) (at 137.16 161.29 0)
+    (property "Value" "2.7pF" (id 1) (at 143.51 140.97 0)
       (effects (font (size 1.27 1.27)) (justify left))
     )
-    (property "Footprint" "Capacitor_SMD:C_0402_1005Metric" (id 2) (at 135.5852 163.83 0)
+    (property "Footprint" "Capacitor_SMD:C_0402_1005Metric" (id 2) (at 141.9352 143.51 0)
       (effects (font (size 1.27 1.27)) hide)
     )
-    (property "Datasheet" "~" (id 3) (at 134.62 160.02 0)
+    (property "Datasheet" "~" (id 3) (at 140.97 139.7 0)
       (effects (font (size 1.27 1.27)) hide)
     )
-    (property "LCSC PN" "" (id 4) (at 134.62 160.02 0)
+    (property "LCSC PN" "" (id 4) (at 140.97 139.7 0)
       (effects (font (size 1.27 1.27)) hide)
     )
@@
     (pin "2")
   )
-  (symbol (lib_id "power:GND") (at 104.14 152.4 0) (unit 1)
+  (symbol (lib_id "power:GND") (at 110.49 132.08 0) (unit 1)
     (in_bom yes) (on_board yes)
-    (property "Reference" "#PWR036" (id 0) (at 104.14 158.75 0)
+    (property "Reference" "#PWR036" (id 0) (at 110.49 138.43 0)
       (effects (font (size 1.27 1.27)) hide)
     )
-    (property "Value" "GND" (id 1) (at 104.14 156.21 0))
-    (property "Footprint" "" (id 2) (at 104.14 152.4 0)
+    (property "Value" "GND" (id 1) (at 110.49 135.89 0))
+    (property "Footprint" "" (id 2) (at 110.49 132.08 0)
       (effects (font (size 1.27 1.27)) hide)
     )
-    (property "Datasheet" "" (id 3) (at 104.14 152.4 0)
+    (property "Datasheet" "" (id 3) (at 110.49 132.08 0)
       (effects (font (size 1.27 1.27)) hide)
     )
@@
     (pin "2")
   )
-  (symbol (lib_id "power:GND") (at 115.57 163.83 0) (unit 1)
+  (symbol (lib_id "power:GND") (at 121.92 143.51 0) (unit 1)
     (in_bom yes) (on_board yes)
-    (property "Reference" "#PWR09" (id 0) (at 115.57 170.18 0)
+    (property "Reference" "#PWR09" (id 0) (at 121.92 149.86 0)
       (effects (font (size 1.27 1.27)) hide)
     )
-    (property "Value" "GND" (id 1) (at 115.57 167.64 0))
-    (property "Footprint" "" (id 2) (at 115.57 163.83 0)
+    (property "Value" "GND" (id 1) (at 121.92 147.32 0))
+    (property "Footprint" "" (id 2) (at 121.92 143.51 0)
       (effects (font (size 1.27 1.27)) hide)
     )
-    (property "Datasheet" "" (id 3) (at 115.57 163.83 0)
+    (property "Datasheet" "" (id 3) (at 121.92 143.51 0)
       (effects (font (size 1.27 1.27)) hide)
     )
@@
     (pin "2")
   )
-  (symbol (lib_id "Device:Antenna_Dipole") (at 106.68 147.32 0) (mirror y) (unit 1)
+  (symbol (lib_id "Device:Antenna_Dipole") (at 113.03 127 0) (mirror y) (unit 1)
     (in_bom yes) (on_board yes)
-    (property "Reference" "AE1" (id 0) (at 106.68 144.78 0)
+    (property "Reference" "AE1" (id 0) (at 113.03 124.46 0)
       (effects (font (size 1.27 1.27)) (justify left))
     )
-    (property "Value" "Antenna_Dipole" (id 1) (at 109.22 147.32 0)
+    (property "Value" "Antenna_Dipole" (id 1) (at 115.57 127 0)
       (effects (font (size 1.27 1.27)) (justify left))
     )
-    (property "Footprint" "RF_Antenna:Texas_SWRA117D_2.4GHz_Right" (id 2) (at 106.68 147.32 0)
+    (property "Footprint" "RF_Antenna:Texas_SWRA117D_2.4GHz_Right" (id 2) (at 113.03 127 0)
       (effects (font (size 1.27 1.27)) hide)
     )
-    (property "Datasheet" "~" (id 3) (at 106.68 147.32 0)
+    (property "Datasheet" "~" (id 3) (at 113.03 127 0)
       (effects (font (size 1.27 1.27)) hide)
     )
@@
     (pin "2")
   )
-  (symbol (lib_id "power:GND") (at 134.62 163.83 0) (unit 1)
+  (symbol (lib_id "power:GND") (at 140.97 143.51 0) (unit 1)
     (in_bom yes) (on_board yes)
-    (property "Reference" "#PWR012" (id 0) (at 134.62 170.18 0)
+    (property "Reference" "#PWR012" (id 0) (at 140.97 149.86 0)
       (effects (font (size 1.27 1.27)) hide)
     )
-    (property "Value" "GND" (id 1) (at 134.62 167.64 0))
-    (property "Footprint" "" (id 2) (at 134.62 163.83 0)
+    (property "Value" "GND" (id 1) (at 140.97 147.32 0))
+    (property "Footprint" "" (id 2) (at 140.97 143.51 0)
       (effects (font (size 1.27 1.27)) hide)
     )
-    (property "Datasheet" "" (id 3) (at 134.62 163.83 0)
+    (property "Datasheet" "" (id 3) (at 140.97 143.51 0)
       (effects (font (size 1.27 1.27)) hide)
     )
@@
     (pin "1")
   )
-  (symbol (lib_id "Device:C") (at 115.57 160.02 0) (unit 1)
+  (symbol (lib_id "Device:C") (at 121.92 139.7 0) (unit 1)
     (in_bom yes) (on_board yes)
-    (property "Reference" "C4" (id 0) (at 118.11 158.75 0)
+    (property "Reference" "C4" (id 0) (at 124.46 138.43 0)
       (effects (font (size 1.27 1.27)) (justify left))
     )
-    (property "Value" "1.0pF" (id 1) (at 118.11 161.29 0)
+    (property "Value" "1.0pF" (id 1) (at 124.46 140.97 0)
       (effects (font (size 1.27 1.27)) (justify left))
     )
-    (property "Footprint" "Capacitor_SMD:C_0402_1005Metric" (id 2) (at 116.5352 163.83 0)
+    (property "Footprint" "Capacitor_SMD:C_0402_1005Metric" (id 2) (at 122.8852 143.51 0)
       (effects (font (size 1.27 1.27)) hide)
     )
-    (property "Datasheet" "~" (id 3) (at 115.57 160.02 0)
+    (property "Datasheet" "~" (id 3) (at 121.92 139.7 0)
       (effects (font (size 1.27 1.27)) hide)
     )
-    (property "LCSC PN" "" (id 4) (at 115.57 160.02 0)
+    (property "LCSC PN" "" (id 4) (at 121.92 139.7 0)
       (effects (font (size 1.27 1.27)) hide)
     )
@@
       (effects (font (size 1.27 1.27)) (justify left))
     )
-    (property "Value" "1N4728A" (id 1) (at 165.1 184.1499 90)
+    (property "Value" "ZM4728A" (id 1) (at 165.1 184.1499 90)
       (effects (font (size 1.27 1.27)) (justify left))
     )
-    (property "Footprint" "Diode_THT:D_DO-41_SOD81_P3.81mm_Vertical_KathodeUp" (id 2) (at 162.56 182.88 0)
+    (property "Footprint" "Diode_SMD:D_MELF" (id 2) (at 162.56 182.88 0)
       (effects (font (size 1.27 1.27)) hide)
     )
@@
       (effects (font (size 1.27 1.27)) hide)
     )
-    (property "LCSC" "C261315" (id 4) (at 162.56 182.88 90)
+    (property "LCSC" "C38989" (id 4) (at 162.56 182.88 90)
       (effects (font (size 1.27 1.27)) hide)
     )
@@
       (effects (font (size 1.27 1.27)) hide)
     )
-    (property "LCSC" "C431541" (id 4) (at 118.11 177.8 0)
+    (property "LCSC" "C319019" (id 4) (at 118.11 177.8 0)
       (effects (font (size 1.27 1.27)) hide)
     )
@@
     )
     (path "/e1e7b798-61ee-4fe8-b9cf-3b74b206974f"
-      (reference "D5") (unit 1) (value "1N4728A") (footprint "Diode_THT:D_DO-41_SOD81_P3.81mm_Vertical_KathodeUp")
+      (reference "D5") (unit 1) (value "ZM4728A") (footprint "Diode_SMD:D_MELF")
     )
     (path "/e9bc74f9-63cc-40ba-b34e-8b8b687517f8"
